File: KiCad/MetalDetector/MetalDetector.kicad_pcb (KiCad board)
At the start: 2 copper layers, 0 parts

Commit message: Inline calibration
Parts:
- added C1: 2.2n, Capacitor_SMD:C_0603_1608Metric_Pad1.08x0.95mm_HandSolder, F.Cu at (57.5, 25.4)
- added C10: 47n, Capacitor_SMD:C_0603_1608Metric_Pad1.08x0.95mm_HandSolder, F.Cu at (234.3, 88.3)
- added C11: 470n, Capacitor_SMD:C_0603_1608Metric_Pad1.08x0.95mm_HandSolder, F.Cu at (57.5, 50.5)
- added C12: 470n, Capacitor_SMD:C_0603_1608Metric_Pad1.08x0.95mm_HandSolder, F.Cu at (57.5, 53.1)
- added C13: 2.2n, Capacitor_SMD:C_0603_1608Metric_Pad1.08x0.95mm_HandSolder, F.Cu at (61.8, 25.4)
- added C14: 330n, Capacitor_SMD:C_1812_4532Metric_Pad1.57x3.40mm_HandSolder, F.Cu at (218.5, 88.3)
- added C15: 330u, Capacitor_SMD:CP_Elec_16x22, F.Cu at (226.3, 67.4)
- added C16: 470n, Capacitor_SMD:C_1206_3216Metric_Pad1.33x1.80mm_HandSolder, F.Cu at (230.1, 84.9)
- added C17: 4.7n, Capacitor_SMD:C_0603_1608Metric_Pad1.08x0.95mm_HandSolder, F.Cu at (61.8, 30.5)
- added C18: 100n, Capacitor_SMD:C_0603_1608Metric_Pad1.08x0.95mm_HandSolder, F.Cu at (61.8, 33.0)
- added C19: 100n, Capacitor_SMD:C_0603_1608Metric_Pad1.08x0.95mm_HandSolder, F.Cu at (61.8, 35.5)
- added C2: 33p, Capacitor_SMD:C_0603_1608Metric_Pad1.08x0.95mm_HandSolder, F.Cu at (57.5, 28.0)
- added C20: 100n, Capacitor_SMD:C_0603_1608Metric_Pad1.08x0.95mm_HandSolder, F.Cu at (61.8, 38.0)
- added C21: 100n, Capacitor_SMD:C_0603_1608Metric_Pad1.08x0.95mm_HandSolder, F.Cu at (61.8, 40.5)
- added C22: 100n, Capacitor_SMD:C_0603_1608Metric_Pad1.08x0.95mm_HandSolder, F.Cu at (61.8, 43.0)
- added C23: 100n, Capacitor_SMD:C_0603_1608Metric_Pad1.08x0.95mm_HandSolder, F.Cu at (61.8, 45.5)
- added C24: 10u, Capacitor_SMD:CP_Elec_5x5.4, F.Cu at (74.2, 97.6)
- added C25: 470n, Capacitor_SMD:C_0603_1608Metric_Pad1.08x0.95mm_HandSolder, F.Cu at (61.8, 48.0)
- added C26: 470n, Capacitor_SMD:C_0603_1608Metric_Pad1.08x0.95mm_HandSolder, F.Cu at (61.8, 50.5)
- added C27: 10u, Capacitor_SMD:CP_Elec_5x5.4, F.Cu at (22.2, 25.2)
- added C28: 47u, Capacitor_SMD:CP_Elec_5x5.4, F.Cu at (22.2, 32.1)
- added C29: 47u, Capacitor_SMD:CP_Elec_5x5.4, F.Cu at (22.2, 38.9)
- added C3: 4.7n, Capacitor_SMD:C_0603_1608Metric_Pad1.08x0.95mm_HandSolder, F.Cu at (57.5, 30.5)
- added C30: 47u, Capacitor_SMD:CP_Elec_5x5.4, F.Cu at (22.2, 45.8)
- added C31: 47u, Capacitor_SMD:CP_Elec_5x5.4, F.Cu at (22.2, 52.6)
- added C32: 100u, Capacitor_SMD:CP_Elec_5x5.4, F.Cu at (22.2, 59.5)
- added C33: 100n, Capacitor_SMD:C_0603_1608Metric_Pad1.08x0.95mm_HandSolder, F.Cu at (61.8, 53.1)
- added C34: 100n, Capacitor_SMD:C_0603_1608Metric_Pad1.08x0.95mm_HandSolder, F.Cu at (66.2, 25.4)
- added C35: 100n, Capacitor_SMD:C_0603_1608Metric_Pad1.08x0.95mm_HandSolder, F.Cu at (66.2, 28.0)
- added C4: 100n, Capacitor_SMD:C_0603_1608Metric_Pad1.08x0.95mm_HandSolder, F.Cu at (57.5, 33.0)
- added C5: 100n, Capacitor_SMD:C_0603_1608Metric_Pad1.08x0.95mm_HandSolder, F.Cu at (57.5, 35.5)
- added C6: 100n, Capacitor_SMD:C_0603_1608Metric_Pad1.08x0.95mm_HandSolder, F.Cu at (57.5, 38.0)
- added C7: C, Capacitor_SMD:C_0603_1608Metric_Pad1.08x0.95mm_HandSolder, F.Cu at (57.5, 40.5)
- added C8: C, Capacitor_SMD:C_0603_1608Metric_Pad1.08x0.95mm_HandSolder, F.Cu at (57.5, 43.0)
- added C9: C, Capacitor_SMD:C_0603_1608Metric_Pad1.08x0.95mm_HandSolder, F.Cu at (57.5, 45.5)
- added D1: 4148, Diode_SMD:D_SOD-323F, F.Cu at (79.9, 98.4)
- added D2: 4148, Diode_SMD:D_SOD-323F, F.Cu at (82.5, 98.4)
- added D3: 4148, Diode_SMD:D_SOD-323F, F.Cu at (28.8, 55.2)
- added D4: 4148, Diode_SMD:D_SOD-323F, F.Cu at (28.8, 58.2)
- added D5: BAT54, Diode_SMD:D_SOD-323F, F.Cu at (28.8, 61.1)
- added D6: BAT54, Diode_SMD:D_SOD-323F, F.Cu at (28.8, 64.1)
- added D7: BAT54, Diode_SMD:D_SOD-323F, F.Cu at (28.8, 67.0)
- added D8: BAT54, Diode_SMD:D_SOD-323F, F.Cu at (28.8, 70.0)
- added JP1: RX_{BAL}, Jumper:SolderJumper-3_P1.3mm_Open_RoundedPad1.0x1.5mm, F.Cu at (88.7, 20.0)
- added JP2: RX_{BAL}, Jumper:SolderJumper-3_P1.3mm_Open_RoundedPad1.0x1.5mm, F.Cu at (88.7, 23.8)
- added JP3: TX_{POL}, Jumper:SolderJumper-3_P1.3mm_Open_RoundedPad1.0x1.5mm, F.Cu at (88.7, 27.7)
- added JP4: RX_{BAL}, Jumper:SolderJumper-3_P1.3mm_Open_RoundedPad1.0x1.5mm, F.Cu at (88.7, 31.5)
- added Q1: BC516, Package_TO_SOT_THT:TO-92, F.Cu at (220.3, 84.0)
- added Q2: BC516, Package_TO_SOT_THT:TO-92, F.Cu at (214.1, 84.0)
- added Q3: BC516, Package_TO_SOT_THT:TO-92, F.Cu at (233.0, 85.3)
- added Q4: BC516, Package_TO_SOT_SMD:SOT-23-3, F.Cu at (52.6, 56.9)
- added Q5: BC517, Package_TO_SOT_SMD:SOT-23-3, F.Cu at (52.6, 61.5)
- added R1: 100k, Resistor_SMD:R_0603_1608Metric_Pad0.98x0.95mm_HandSolder, F.Cu at (66.2, 30.5)
- added R10: 10k, Resistor_SMD:R_0603_1608Metric_Pad0.98x0.95mm_HandSolder, F.Cu at (66.2, 48.0)
- added R11: 1k, Resistor_SMD:R_0603_1608Metric_Pad0.98x0.95mm_HandSolder, F.Cu at (66.2, 50.5)
- added R12: 100k, Resistor_SMD:R_0603_1608Metric_Pad0.98x0.95mm_HandSolder, F.Cu at (66.2, 53.1)
- added R13: 56k, Resistor_SMD:R_0603_1608Metric_Pad0.98x0.95mm_HandSolder, F.Cu at (215.4, 80.2)
- added R14: 56k, Resistor_SMD:R_0603_1608Metric_Pad0.98x0.95mm_HandSolder, F.Cu at (215.4, 78.5)
- added R15: 22k, Resistor_SMD:R_0603_1608Metric_Pad0.98x0.95mm_HandSolder, F.Cu at (231.4, 80.5)
- added R16: 10K, Resistor_SMD:R_0603_1608Metric_Pad0.98x0.95mm_HandSolder, F.Cu at (70.5, 33.0)
- added R17: 47k, Resistor_SMD:R_0603_1608Metric_Pad0.98x0.95mm_HandSolder, F.Cu at (70.5, 35.5)
- added R18: 10k, Resistor_SMD:R_0603_1608Metric_Pad0.98x0.95mm_HandSolder, F.Cu at (70.5, 38.0)
- added R19: 100k, Resistor_SMD:R_0603_1608Metric_Pad0.98x0.95mm_HandSolder, F.Cu at (70.5, 40.5)
- added R2: 220, Resistor_SMD:R_1206_3216Metric_Pad1.30x1.75mm_HandSolder, F.Cu at (221.6, 79.3)
- added R20: 4.7k, Resistor_SMD:R_0603_1608Metric_Pad0.98x0.95mm_HandSolder, F.Cu at (70.5, 43.0)
- added R21: 4.7k, Resistor_SMD:R_0603_1608Metric_Pad0.98x0.95mm_HandSolder, F.Cu at (70.5, 45.5)
- added R22: 1M, Resistor_SMD:R_0603_1608Metric_Pad0.98x0.95mm_HandSolder, F.Cu at (82.5, 95.6)
- added R23: 4.7k, Resistor_SMD:R_0603_1608Metric_Pad0.98x0.95mm_HandSolder, F.Cu at (82.5, 93.9)
- added R24: 10k, Resistor_SMD:R_0603_1608Metric_Pad0.98x0.95mm_HandSolder, F.Cu at (70.5, 53.1)
- added R25: 10k, Resistor_SMD:R_0603_1608Metric_Pad0.98x0.95mm_HandSolder, F.Cu at (74.9, 25.4)
- added R26: 22k, Resistor_SMD:R_0603_1608Metric_Pad0.98x0.95mm_HandSolder, F.Cu at (79.0, 95.6)
- added R27: 1M, Resistor_SMD:R_0603_1608Metric_Pad0.98x0.95mm_HandSolder, F.Cu at (74.9, 30.5)
- added R28: 4.7k, Resistor_SMD:R_0603_1608Metric_Pad0.98x0.95mm_HandSolder, F.Cu at (74.9, 33.0)
- added R29: 22k, Resistor_SMD:R_0603_1608Metric_Pad0.98x0.95mm_HandSolder, F.Cu at (74.9, 35.5)
- added R3: 4.7k, Resistor_SMD:R_0603_1608Metric_Pad0.98x0.95mm_HandSolder, F.Cu at (66.2, 33.0)
- added R30: 47k, Resistor_SMD:R_0603_1608Metric_Pad0.98x0.95mm_HandSolder, F.Cu at (74.9, 38.0)
- added R31: 4k7, Resistor_SMD:R_0603_1608Metric_Pad0.98x0.95mm_HandSolder, F.Cu at (74.9, 40.5)
- added R32: 56k, Resistor_SMD:R_0603_1608Metric_Pad0.98x0.95mm_HandSolder, F.Cu at (74.9, 43.0)
- added R33: 4.7k, Resistor_SMD:R_0603_1608Metric_Pad0.98x0.95mm_HandSolder, F.Cu at (74.9, 45.5)
- added R34: 2.2k, Resistor_SMD:R_0603_1608Metric_Pad0.98x0.95mm_HandSolder, F.Cu at (74.9, 48.0)
- added R35: 56k, Resistor_SMD:R_0603_1608Metric_Pad0.98x0.95mm_HandSolder, F.Cu at (74.9, 50.5)
- added R36: 10k, Resistor_SMD:R_0603_1608Metric_Pad0.98x0.95mm_HandSolder, F.Cu at (74.9, 53.1)
- added R37: 4k7, Resistor_SMD:R_0603_1608Metric_Pad0.98x0.95mm_HandSolder, F.Cu at (79.2, 25.4)
- added R38: 2.2k, Resistor_SMD:R_0603_1608Metric_Pad0.98x0.95mm_HandSolder, F.Cu at (79.2, 28.0)
- added R39: 47k, Resistor_SMD:R_0603_1608Metric_Pad0.98x0.95mm_HandSolder, F.Cu at (79.2, 30.5)
- added R4: 100k, Resistor_SMD:R_0603_1608Metric_Pad0.98x0.95mm_HandSolder, F.Cu at (66.2, 35.5)
- added R40: 18k, Resistor_SMD:R_0603_1608Metric_Pad0.98x0.95mm_HandSolder, F.Cu at (79.2, 33.0)
- added R41: 4.7k, Resistor_SMD:R_0603_1608Metric_Pad0.98x0.95mm_HandSolder, F.Cu at (79.2, 35.5)
- added R42: 4.7k, Resistor_SMD:R_0603_1608Metric_Pad0.98x0.95mm_HandSolder, F.Cu at (79.2, 38.0)
- added R43: 10k, Resistor_SMD:R_0603_1608Metric_Pad0.98x0.95mm_HandSolder, F.Cu at (79.2, 40.5)
- added R44: 10k, Resistor_SMD:R_0603_1608Metric_Pad0.98x0.95mm_HandSolder, F.Cu at (79.2, 43.0)
- added R45: 4.7k, Resistor_SMD:R_0603_1608Metric_Pad0.98x0.95mm_HandSolder, F.Cu at (79.2, 45.5)
- added R46: 10k, Resistor_SMD:R_0603_1608Metric_Pad0.98x0.95mm_HandSolder, F.Cu at (79.2, 48.0)
- added R47: 10k, Resistor_SMD:R_0603_1608Metric_Pad0.98x0.95mm_HandSolder, F.Cu at (79.2, 50.5)
- added R5: 12k, Resistor_SMD:R_0603_1608Metric_Pad0.98x0.95mm_HandSolder, F.Cu at (231.4, 78.8)
- added R6: 1k, Resistor_SMD:R_1206_3216Metric_Pad1.30x1.75mm_HandSolder, F.Cu at (235.6, 79.0)
- added R7: 47k, Resistor_SMD:R_0603_1608Metric_Pad0.98x0.95mm_HandSolder, F.Cu at (66.2, 40.5)
- added R8: 1k, Resistor_SMD:R_0603_1608Metric_Pad0.98x0.95mm_HandSolder, F.Cu at (66.2, 43.0)
- added R9: 10k, Resistor_SMD:R_0603_1608Metric_Pad0.98x0.95mm_HandSolder, F.Cu at (66.2, 45.5)
- added RV1: 47k, Potentiometer_SMD:Potentiometer_Bourns_3269W_Vertical, F.Cu at (39.1, 19.6)
- added RV2: 100k, Potentiometer_SMD:Potentiometer_Bourns_3269W_Vertical, F.Cu at (47.0, 19.6)
- added RV3: 47k, Potentiometer_SMD:Potentiometer_Bourns_3269W_Vertical, F.Cu at (55.0, 19.6)
- added RV4: 100k, Potentiometer_SMD:Potentiometer_Bourns_3269W_Vertical, F.Cu at (62.9, 19.6)
- added TP1: BAL_{CROSS}, TestPoint:TestPoint_Keystone_5010-5014_Multipurpose, F.Cu at (37.6, 26.7)
- added TP10: TX_{+}, TestPoint:TestPoint_Keystone_5010-5014_Multipurpose, F.Cu at (42.7, 41.9)
- added TP11: Q_{SYNC}, TestPoint:TestPoint_Keystone_5010-5014_Multipurpose, F.Cu at (42.7, 46.9)
- added TP12: BAL_{COLPITTS}, TestPoint:TestPoint_Keystone_5010-5014_Multipurpose, F.Cu at (42.7, 52.0)
- added TP13: G_{SYNC}, TestPoint:TestPoint_Keystone_5010-5014_Multipurpose, F.Cu at (47.7, 26.7)
- added TP14: RX_{N}, TestPoint:TestPoint_Keystone_5010-5014_Multipurpose, F.Cu at (47.7, 31.8)
- added TP15: Q, TestPoint:TestPoint_Keystone_5010-5014_Multipurpose, F.Cu at (47.7, 36.8)
- added TP16: TX_{SYNC}, TestPoint:TestPoint_Keystone_5010-5014_Multipurpose, F.Cu at (47.7, 41.9)
- added TP17: Q_{BIAS}, TestPoint:TestPoint_Keystone_5010-5014_Multipurpose, F.Cu at (47.7, 46.9)
- added TP18: ADC_{BIAS}, TestPoint:TestPoint_Keystone_5010-5014_Multipurpose, F.Cu at (47.7, 52.0)
- added TP19: Vee, TestPoint:TestPoint_Keystone_5010-5014_Multipurpose, F.Cu at (52.8, 26.7)
- added TP2: I, TestPoint:TestPoint_Keystone_5010-5014_Multipurpose, F.Cu at (37.6, 31.8)
- added TP20: I_{ADC}, TestPoint:TestPoint_Keystone_5010-5014_Multipurpose, F.Cu at (52.8, 31.8)
- added TP21: Q_{ADC}, TestPoint:TestPoint_Keystone_5010-5014_Multipurpose, F.Cu at (52.8, 36.8)
- added TP3: RX_{P}, TestPoint:TestPoint_Keystone_5010-5014_Multipurpose, F.Cu at (37.6, 36.8)
- added TP4: I_{CLK}, TestPoint:TestPoint_Keystone_5010-5014_Multipurpose, F.Cu at (37.6, 41.9)
- added TP5: Q_{CLK}, TestPoint:TestPoint_Keystone_5010-5014_Multipurpose, F.Cu at (37.6, 46.9)
- added TP6: TX_{COLPITTS}, TestPoint:TestPoint_Keystone_5010-5014_Multipurpose, F.Cu at (37.6, 52.0)
- added TP7: G_{CLK}, TestPoint:TestPoint_Keystone_5010-5014_Multipurpose, F.Cu at (42.7, 26.7)
- added TP8: I_{SYNC}, TestPoint:TestPoint_Keystone_5010-5014_Multipurpose, F.Cu at (42.7, 31.8)
- added TP9: TX_{-}, TestPoint:TestPoint_Keystone_5010-5014_Multipurpose, F.Cu at (42.7, 36.8)
- added U1: NE5532, Package_SO:SOIC-8_3.9x4.9mm_P1.27mm, F.Cu at (30.9, 18.3)
- added U2: NE5532, Package_SO:SOIC-8_3.9x4.9mm_P1.27mm, F.Cu at (30.9, 24.9)
- added U3: CD4053B, Package_SO:SOIC-16_3.9x9.9mm_P1.27mm, F.Cu at (45.8, 60.4)
- added U4: LM393, Package_SO:SOIC-8_3.9x4.9mm_P1.27mm, F.Cu at (88.3, 97.5)
- added U5: NE5532, Package_SO:SOIC-8_3.9x4.9mm_P1.27mm, F.Cu at (30.9, 38.0)
- added U6: TS912, Package_SO:SOIC-8_3.9x4.9mm_P1.27mm, F.Cu at (30.9, 44.6)
Routing:
- net /TX_{+}: track 0.00 -> 14.6 mm
- net Net-(Q1-E): track 0.00 -> 13.7 mm
- net /TX_{-}: track 0.00 -> 10.7 mm
- net Net-(Q1-B): track 0.00 -> 8.32 mm
- net /TX_{COLPITTS}: track 0.00 -> 8.04 mm
- net Net-(Q3-E): track 0.00 -> 7.99 mm
- net Net-(Q3-B): track 0.00 -> 6.55 mm
- net VCC: track 0.00 -> 6.03 mm
- net Net-(Q2-B): track 0.00 -> 2.95 mm
Other:
- board outline added: 100 x 50 mm
- copper layers 2 -> 4
