File: KiCad/MetalDetector/MetalDetector.kicad_sch (KiCad schematic)
At the start: 138 parts, among them J1 TX COILS, J2 RX, J3 SYNC, J4 BATTERY, J5 CHARGE PUMP, J6 SYNC, Q1 BC516, Q2 BC516, Q3 BC516, Q4 BC516, Q5 BC517, U1 NE5532, U2 LM393, U3 MC33063AP, U4 MC33063AP, U5 TS912, U6 NE5532, U7 NE5532, U8 CD4053B

Commit message: Push
Added test points to schematic
Parts:
- removed C17, C20: 330u, Capacitor_THT:CP_Radial_D8.0mm_P5.00mm, symbol Device:C_Polarized
- removed C18, C22: 100u, Capacitor_THT:CP_Radial_D8.0mm_P5.00mm, symbol Device:C_Polarized
- removed C19: 470p, Capacitor_THT:C_Disc_D6.0mm_W2.5mm_P5.00mm, symbol Device:C
- removed C21: 1500p, Capacitor_THT:C_Disc_D6.0mm_W2.5mm_P5.00mm, symbol Device:C
- removed D5, D6: 1N5819, Diode_THT:D_DO-41_SOD81_P10.16mm_Horizontal, symbol Diode:1N5819
- removed J6: SYNC, Connector_PinHeader_2.54mm:PinHeader_1x06_P2.54mm_Vertical, symbol Connector_Generic:Conn_01x06
- removed JP5: SUPPLY, Jumper:SolderJumper-3_P1.3mm_Open_RoundedPad1.0x1.5mm, symbol Jumper:SolderJumper_3_Open
- removed L5, L6: 330u, Inductor_THT:L_Radial_D6.0mm_P4.00mm, symbol Device:L_Ferrite
- removed R22: 0.33, Resistor_THT:R_Axial_DIN0207_L6.3mm_D2.5mm_P10.16mm_Horizontal, symbol Device:R
- removed R23: 180, Resistor_THT:R_Axial_DIN0207_L6.3mm_D2.5mm_P10.16mm_Horizontal, symbol Device:R
- removed R24: 0.22, Resistor_THT:R_Axial_DIN0207_L6.3mm_D2.5mm_P10.16mm_Horizontal, symbol Device:R
- removed R25, R26, R27, R28: R, Resistor_THT:R_Axial_DIN0207_L6.3mm_D2.5mm_P10.16mm_Horizontal, symbol Device:R
- removed U3, U4: MC33063AP, Package_DIP:DIP-8_W7.62mm_Socket, symbol Regulator_Switching:MC33063AP
- added C?: 330u, symbol Device:C_Polarized
- added J?: ADC, symbol Connector_Generic:Conn_01x03
- added J?: CLOCKS, symbol Connector_Generic:Conn_01x03
- added J?: OSC_{SUPLLY}, symbol Connector_Generic:Conn_01x02
- added TP1: TX_{-}, symbol Connector:TestPoint_Small
- added TP10: Q_{CLK}, symbol Connector:TestPoint_Small
- added TP11: G_{CLK}, symbol Connector:TestPoint_Small
- added TP12: I_{SYNC}, symbol Connector:TestPoint_Small
- added TP13: Q_{SYNC}, symbol Connector:TestPoint_Small
- added TP14: G_{SYNC}, symbol Connector:TestPoint_Small
- added TP15: I, symbol Connector:TestPoint_Small
- added TP16: Q, symbol Connector:TestPoint_Small
- added TP17: ADC_{BIAS}, symbol Connector:TestPoint_Small
- added TP18: Q_{BIAS}, symbol Connector:TestPoint_Small
- added TP19: I_{ADC}, symbol Connector:TestPoint_Small
- added TP2: TX_{COLPITTS}, symbol Connector:TestPoint_Small
- added TP20: Q_{ADC}, symbol Connector:TestPoint_Small
- added TP3: BAL_{CROSS}, symbol Connector:TestPoint_Small
- added TP4: BAL_{COLPITTS}, symbol Connector:TestPoint_Small
- added TP5: RX_{P}, symbol Connector:TestPoint_Small
- added TP6: RX_{N}, symbol Connector:TestPoint_Small
- added TP7: TX_{SYNC}, symbol Connector:TestPoint_Small
- added TP8: Vee, symbol Connector:TestPoint_Small
- added TP9: I_{CLK}, symbol Connector:TestPoint_Small
- added TP?: TX_{+}, symbol Connector:TestPoint_Small
- C1: renamed from C2; footprint Capacitor_THT:C_Disc_D6.0mm_W2.5mm_P5.00mm -> (none)
- C10: renamed from C7; footprint Capacitor_THT:C_Disc_D6.0mm_W2.5mm_P5.00mm -> (none)
- C11: renamed from C32; footprint Capacitor_THT:C_Disc_D6.0mm_W4.4mm_P5.00mm -> (none)
- C12: renamed from C33; footprint Capacitor_THT:C_Disc_D6.0mm_W4.4mm_P5.00mm -> (none)
- C13: renamed from C12; footprint Capacitor_THT:C_Disc_D6.0mm_W2.5mm_P5.00mm -> (none)
- C14: renamed from C8; footprint Capacitor_THT:C_Disc_D6.0mm_W4.4mm_P5.00mm -> (none)
- C15: renamed from C9; footprint Capacitor_THT:C_Disc_D6.0mm_W4.4mm_P5.00mm -> (none)
- C16: renamed from C35; footprint Capacitor_THT:C_Disc_D6.0mm_W2.5mm_P5.00mm -> (none)
- C17: renamed from C36; footprint Capacitor_THT:C_Disc_D6.0mm_W2.5mm_P5.00mm -> (none)
- C18: renamed from C13; footprint Capacitor_THT:C_Disc_D6.0mm_W2.5mm_P5.00mm -> (none)
- C19: renamed from C10; footprint Capacitor_THT:C_Disc_D6.0mm_W2.5mm_P5.00mm -> (none)
- C2: renamed from C1; footprint Capacitor_THT:C_Disc_D6.0mm_W2.5mm_P5.00mm -> (none)
- C20: renamed from C11; footprint Capacitor_THT:C_Disc_D6.0mm_W2.5mm_P5.00mm -> (none)
- C21: renamed from C39; footprint Capacitor_THT:C_Disc_D6.0mm_W2.5mm_P5.00mm -> (none)
- C22: renamed from C40; footprint Capacitor_THT:C_Disc_D6.0mm_W2.5mm_P5.00mm -> (none)
- C23: renamed from C34; footprint Capacitor_THT:C_Disc_D6.0mm_W2.5mm_P5.00mm -> (none)
- C24: renamed from C14; footprint Capacitor_THT:C_Disc_D6.0mm_W2.5mm_P5.00mm -> (none)
- C25: renamed from C15; footprint Capacitor_THT:CP_Radial_D4.0mm_P2.00mm -> (none)
- C26: renamed from C37; footprint Capacitor_THT:C_Disc_D6.0mm_W4.4mm_P5.00mm -> (none)
- C27: renamed from C38; footprint Capacitor_THT:C_Disc_D6.0mm_W4.4mm_P5.00mm -> (none)
- C28: renamed from C16; footprint Capacitor_THT:CP_Radial_D4.0mm_P2.00mm -> (none)
- C29: renamed from C23; footprint Capacitor_THT:CP_Radial_D8.0mm_P5.00mm -> (none)
- C3: footprint Capacitor_THT:C_Disc_D6.0mm_W2.5mm_P5.00mm -> (none)
- C30: renamed from C24; footprint Capacitor_THT:CP_Radial_D8.0mm_P5.00mm -> (none)
- C31: renamed from C25; footprint Capacitor_THT:CP_Radial_D8.0mm_P5.00mm -> (none)
- C32: renamed from C26; footprint Capacitor_THT:CP_Radial_D8.0mm_P5.00mm -> (none)
- C34: renamed from C30; footprint Capacitor_THT:C_Disc_D6.0mm_W2.5mm_P5.00mm -> (none)
- C4: renamed from C27; footprint Capacitor_THT:C_Disc_D6.0mm_W2.5mm_P5.00mm -> (none)
- C5: renamed from C28; footprint Capacitor_THT:C_Disc_D6.0mm_W2.5mm_P5.00mm -> (none)
- C6: renamed from C29; footprint Capacitor_THT:C_Disc_D6.0mm_W2.5mm_P5.00mm -> (none)
- C7: renamed from C4; footprint Capacitor_THT:C_Disc_D6.0mm_W2.5mm_P5.00mm -> (none)
- C8: renamed from C5; footprint Capacitor_THT:C_Disc_D6.0mm_W2.5mm_P5.00mm -> (none)
- C9: renamed from C6; footprint Capacitor_THT:C_Disc_D6.0mm_W2.5mm_P5.00mm -> (none)
- D1, D2, D3, D4: footprint Diode_THT:D_DO-35_SOD27_P7.62mm_Horizontal -> (none)
- D5: renamed from D7; footprint Diode_THT:D_DO-35_SOD27_P7.62mm_Horizontal -> (none)
- D6: renamed from D8; footprint Diode_THT:D_DO-35_SOD27_P7.62mm_Horizontal -> (none)
- D7: renamed from D9; footprint Diode_THT:D_DO-35_SOD27_P7.62mm_Horizontal -> (none)
- D8: renamed from D10; footprint Diode_THT:D_DO-35_SOD27_P7.62mm_Horizontal -> (none)
- J1: footprint Connector_PinHeader_2.54mm:PinHeader_1x05_P2.54mm_Vertical -> (none)
- J2: footprint Connector_PinHeader_2.54mm:PinHeader_1x03_P2.54mm_Vertical -> (none)
- J4: renamed from J5; footprint Connector_PinHeader_2.54mm:PinHeader_1x03_P2.54mm_Vertical -> (none)
- J5: renamed from J3; footprint Connector_PinHeader_2.54mm:PinHeader_1x03_P2.54mm_Vertical -> (none)
- J6: renamed from J4; footprint Connector_PinHeader_2.54mm:PinHeader_1x02_P2.54mm_Vertical -> (none)
- JP1, JP2, JP3, JP4: footprint Jumper:SolderJumper-3_P1.3mm_Open_RoundedPad1.0x1.5mm -> (none)
- Q1, Q2, Q3, Q4, Q5: footprint Package_TO_SOT_THT:TO-92_Inline -> (none)
- R1: renamed from R33; footprint Resistor_THT:R_Axial_DIN0207_L6.3mm_D2.5mm_P10.16mm_Horizontal -> (none)
- R10: renamed from R36; footprint Resistor_THT:R_Axial_DIN0207_L6.3mm_D2.5mm_P10.16mm_Horizontal -> (none)
- R11: renamed from R6; footprint Resistor_THT:R_Axial_DIN0207_L6.3mm_D2.5mm_P10.16mm_Horizontal -> (none)
- R12: renamed from R10; footprint Resistor_THT:R_Axial_DIN0207_L6.3mm_D2.5mm_P10.16mm_Horizontal -> (none)
- R13: renamed from R8; footprint Resistor_THT:R_Axial_DIN0207_L6.3mm_D2.5mm_P10.16mm_Horizontal -> (none)
- R14: renamed from R9; footprint Resistor_THT:R_Axial_DIN0207_L6.3mm_D2.5mm_P10.16mm_Horizontal -> (none)
- R15: renamed from R11; footprint Resistor_THT:R_Axial_DIN0207_L6.3mm_D2.5mm_P10.16mm_Horizontal -> (none)
- R16: renamed from R12; footprint Resistor_THT:R_Axial_DIN0207_L6.3mm_D2.5mm_P10.16mm_Horizontal -> (none)
- R17: renamed from R15; footprint Resistor_THT:R_Axial_DIN0207_L6.3mm_D2.5mm_P10.16mm_Horizontal -> (none)
- R18: renamed from R13; footprint Resistor_THT:R_Axial_DIN0207_L6.3mm_D2.5mm_P10.16mm_Horizontal -> (none)
- R19: renamed from R37; footprint Resistor_THT:R_Axial_DIN0207_L6.3mm_D2.5mm_P10.16mm_Horizontal -> (none)
- R2: renamed from R1; footprint Resistor_THT:R_Axial_DIN0207_L6.3mm_D2.5mm_P10.16mm_Horizontal -> (none)
- R20: renamed from R14; footprint Resistor_THT:R_Axial_DIN0207_L6.3mm_D2.5mm_P10.16mm_Horizontal -> (none)
- R21: renamed from R39; footprint Resistor_THT:R_Axial_DIN0207_L6.3mm_D2.5mm_P10.16mm_Horizontal -> (none)
- R22: renamed from R16; footprint Resistor_THT:R_Axial_DIN0207_L6.3mm_D2.5mm_P10.16mm_Horizontal -> (none)
- R23: renamed from R17; footprint Resistor_THT:R_Axial_DIN0207_L6.3mm_D2.5mm_P10.16mm_Horizontal -> (none)
- R24: renamed from R42; footprint Resistor_THT:R_Axial_DIN0207_L6.3mm_D2.5mm_P10.16mm_Horizontal -> (none)
- R25: renamed from R43; footprint Resistor_THT:R_Axial_DIN0207_L6.3mm_D2.5mm_P10.16mm_Horizontal -> (none)
- R26: renamed from R18; footprint Resistor_THT:R_Axial_DIN0207_L6.3mm_D2.5mm_P10.16mm_Horizontal -> (none)
- R27: renamed from R19; footprint Resistor_THT:R_Axial_DIN0207_L6.3mm_D2.5mm_P10.16mm_Horizontal -> (none)
- R28: renamed from R20; footprint Resistor_THT:R_Axial_DIN0207_L6.3mm_D2.5mm_P10.16mm_Horizontal -> (none)
- R29: renamed from R21; footprint Resistor_THT:R_Axial_DIN0207_L6.3mm_D2.5mm_P10.16mm_Horizontal -> (none)
- R3: renamed from R34; footprint Resistor_THT:R_Axial_DIN0207_L6.3mm_D2.5mm_P10.16mm_Horizontal -> (none)
- R30: renamed from R29; footprint Resistor_THT:R_Axial_DIN0207_L6.3mm_D2.5mm_P10.16mm_Horizontal -> (none)
- R31: renamed from R30; footprint Resistor_THT:R_Axial_DIN0207_L6.3mm_D2.5mm_P10.16mm_Horizontal -> (none)
- R37: renamed from R31; footprint Resistor_THT:R_Axial_DIN0207_L6.3mm_D2.5mm_P10.16mm_Horizontal -> (none)
- R39: renamed from R32; footprint Resistor_THT:R_Axial_DIN0207_L6.3mm_D2.5mm_P10.16mm_Horizontal -> (none)
- R4: renamed from R2; footprint Resistor_THT:R_Axial_DIN0207_L6.3mm_D2.5mm_P10.16mm_Horizontal -> (none)
- R5: renamed from R3; footprint Resistor_THT:R_Axial_DIN0207_L6.3mm_D2.5mm_P10.16mm_Horizontal -> (none)
- R6: renamed from R4; footprint Resistor_THT:R_Axial_DIN0207_L6.3mm_D2.5mm_P10.16mm_Horizontal -> (none)
- R7: footprint Resistor_THT:R_Axial_DIN0207_L6.3mm_D2.5mm_P10.16mm_Horizontal -> (none)
- R8: renamed from R5; footprint Resistor_THT:R_Axial_DIN0207_L6.3mm_D2.5mm_P10.16mm_Horizontal -> (none)
- R9: renamed from R35; footprint Resistor_THT:R_Axial_DIN0207_L6.3mm_D2.5mm_P10.16mm_Horizontal -> (none)
- RV1, RV2, RV3, RV4: footprint Potentiometer_THT:Potentiometer_Bourns_3266Y_Vertical -> (none)
- U1: renamed from U6; footprint Package_DIP:DIP-8_W7.62mm_Socket -> (none)
- U2: renamed from U7; footprint Package_DIP:DIP-8_W7.62mm_Socket -> (none)
- U3: renamed from U1; footprint Package_DIP:DIP-8_W7.62mm_Socket -> (none)
- U4: renamed from U8; footprint Package_DIP:DIP-16_W7.62mm_Socket -> (none)
- U5: renamed from U2; footprint Package_DIP:DIP-8_W7.62mm_Socket -> (none)
- gave numbers to parts that had none: 4
- renumbered C41 to C33, R50 to R35, R48 to R36, R47 to R38, R49 to R41, R38 to R42, R40 to R43, R41 to R44, R44 to R45, R45 to R46, R46 to R47, U5 to U6
Connections:
- net -5V: now also TP8.1
- net GND: now also C?.2, J?.2 (Pin_2), J?.2 (Pin_2)
- net G_{CLK}: now also TP11.1
- net G_{SYNC}: now also TP14.1
- net I: now also TP15.1
- net I_{ADC}: now also J?.1 (Pin_1), TP19.1
- net I_{CLK}: now also TP9.1
- net I_{SYNC}: now also TP12.1
- net Q: now also TP16.1
- net Q_{ADC}: now also J?.3 (Pin_3), TP20.1
- net Q_{CLK}: now also TP10.1
- net Q_{SYNC}: now also TP13.1
- net RX_{N}: now also TP6.1
- net RX_{P}: now also TP5.1
- net TX_{+}: now also TP?.1
- net TX_{-}: now also TP1.1
- net TX_{COLPITTS}: now also TP2.1
- net TX_{SYNC}: now also TP7.1
- net VCC: now also C?.1, J?.1 (Pin_1)
- net V_{BIAS-}: now also TP18.1; no longer R21.2
- net at JP1.2 (C), R7.2: now also TP3.1
- net at JP2.2 (C), R17.2: now also TP4.1
- net V_{BIAS+} renamed ADC_{BIAS}
- net ADC_{BIAS}: now also TP17.1
- new net G_CLK: J?.3 (Pin_3)
- new net I_CLK: J?.1 (Pin_1)
- new net Q_CLK: J?.2 (Pin_2)
- new net Q_{BIAS}: R21.2
Other:
- note added: "As mentioned above, the Q signal is actually the one that samples the RX signal in phase. It is a strong signal when no target is present, it lowers when a meaningfull target is present and rises when the target is ferrous. It needs bias to be set to 0 when no target are present, so that the biggest output swing dinamic is achived."
- note removed: "As mentioned above, the Q signal is actually the one that samples the RX signal in phase. It is a strong signal when no target is present, it lowers when a meaningfull target is present and rises when the target is ferrous. In needs bias to be set to 0 when no target are present, so that the biggest output swing dinamic is achived."
- note removed: "Experiment not implemented: I want to see what happends if I drive the oscillator at something like 25V or more. This is a boost converter"
- note removed: "Unimplemented: for now I am using the NUCLEO dev board to provide both 3.3V and 5V."
- moved on the sheet: C1, C13, C16, C17, C18, C29, C3, C30, C31, C32, C34, D5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

Commit message: Push
Kicad footprint assignment
Parts:
- C1, C10, C11, C12, C13, C2, C3, C4, C5, C6, C7, C8, C9: footprint (none) -> Capacitor_SMD:C_0603_1608Metric_Pad1.08x0.95mm_HandSolder
- C14: footprint (none) -> Capacitor_SMD:C_1812_4532Metric_Pad1.57x3.40mm_HandSolder
- C15: renamed from C?; footprint (none) -> Capacitor_SMD:CP_Elec_16x22
- C16: renamed from C15; footprint (none) -> Capacitor_SMD:C_0603_1608Metric_Pad1.08x0.95mm_HandSolder
- C17: renamed from C18; footprint (none) -> Capacitor_SMD:C_0603_1608Metric_Pad1.08x0.95mm_HandSolder
- C18: renamed from C19; footprint (none) -> Capacitor_SMD:C_0603_1608Metric_Pad1.08x0.95mm_HandSolder
- C19: renamed from C20; footprint (none) -> Capacitor_SMD:C_0603_1608Metric_Pad1.08x0.95mm_HandSolder
- C20: renamed from C21; footprint (none) -> Capacitor_SMD:C_0603_1608Metric_Pad1.08x0.95mm_HandSolder
- C21: renamed from C22; footprint (none) -> Capacitor_SMD:C_0603_1608Metric_Pad1.08x0.95mm_HandSolder
- C22: renamed from C23; footprint (none) -> Capacitor_SMD:C_0603_1608Metric_Pad1.08x0.95mm_HandSolder
- C23: renamed from C24; footprint (none) -> Capacitor_SMD:C_0603_1608Metric_Pad1.08x0.95mm_HandSolder
- C24: renamed from C25; footprint (none) -> Capacitor_SMD:CP_Elec_5x5.4
- C25: renamed from C26; footprint (none) -> Capacitor_SMD:C_0603_1608Metric_Pad1.08x0.95mm_HandSolder
- C26: renamed from C27; footprint (none) -> Capacitor_SMD:C_0603_1608Metric_Pad1.08x0.95mm_HandSolder
- C27: renamed from C28; footprint (none) -> Capacitor_SMD:CP_Elec_5x5.4
- C28: renamed from C29; footprint (none) -> Capacitor_SMD:CP_Elec_5x5.4
- C29: renamed from C30; footprint (none) -> Capacitor_SMD:CP_Elec_5x5.4
- C30: renamed from C31; footprint (none) -> Capacitor_SMD:CP_Elec_5x5.4
- C31: renamed from C32; footprint (none) -> Capacitor_SMD:CP_Elec_5x5.4
- C32: renamed from C33; footprint (none) -> Capacitor_SMD:CP_Elec_5x5.4
- C33: renamed from C16; footprint (none) -> Capacitor_SMD:C_0603_1608Metric_Pad1.08x0.95mm_HandSolder
- C34: renamed from C17; footprint (none) -> Capacitor_SMD:C_0603_1608Metric_Pad1.08x0.95mm_HandSolder
- C35: renamed from C34; footprint (none) -> Capacitor_SMD:C_0603_1608Metric_Pad1.08x0.95mm_HandSolder
- D1, D2, D3, D4, D5, D6, D7, D8: footprint (none) -> Diode_SMD:D_SOD-323F
- Q1, Q2, Q3: footprint (none) -> Package_TO_SOT_THT:TO-92
- Q4, Q5: footprint (none) -> Package_TO_SOT_SMD:SOT-23-3
- R1, R10, R11, R12, R13, R14, R15, R16, R17, R18, R19, R20, R21, R22, R23, R24, R25, R26, R27, R28, R29, R3, R30, R31, R32, R33, R34, R35, R36, R37, R38, R39, R4, R40, R41, R42, R43, R44, R45, R46, R47, R5, R7, R8, R9: footprint (none) -> Resistor_SMD:R_0603_1608Metric_Pad0.98x0.95mm_HandSolder
- R2, R6: footprint (none) -> Resistor_SMD:R_1206_3216Metric_Pad1.30x1.75mm_HandSolder
- TP1: renamed from TP3; footprint (none) -> TestPoint:TestPoint_Keystone_5010-5014_Multipurpose
- TP10: renamed from TP?; footprint (none) -> TestPoint:TestPoint_Keystone_5010-5014_Multipurpose
- TP11: renamed from TP13; footprint (none) -> TestPoint:TestPoint_Keystone_5010-5014_Multipurpose
- TP12: renamed from TP4; footprint (none) -> TestPoint:TestPoint_Keystone_5010-5014_Multipurpose
- TP13: renamed from TP14; footprint (none) -> TestPoint:TestPoint_Keystone_5010-5014_Multipurpose
- TP14: renamed from TP6; footprint (none) -> TestPoint:TestPoint_Keystone_5010-5014_Multipurpose
- TP15: renamed from TP16; footprint (none) -> TestPoint:TestPoint_Keystone_5010-5014_Multipurpose
- TP16: renamed from TP7; footprint (none) -> TestPoint:TestPoint_Keystone_5010-5014_Multipurpose
- TP17: renamed from TP18; footprint (none) -> TestPoint:TestPoint_Keystone_5010-5014_Multipurpose
- TP18: renamed from TP17; footprint (none) -> TestPoint:TestPoint_Keystone_5010-5014_Multipurpose
- TP19: renamed from TP8; footprint (none) -> TestPoint:TestPoint_Keystone_5010-5014_Multipurpose
- TP2: renamed from TP15; footprint (none) -> TestPoint:TestPoint_Keystone_5010-5014_Multipurpose
- TP20: renamed from TP19; footprint (none) -> TestPoint:TestPoint_Keystone_5010-5014_Multipurpose
- TP21: renamed from TP20; footprint (none) -> TestPoint:TestPoint_Keystone_5010-5014_Multipurpose
- TP3: renamed from TP5; footprint (none) -> TestPoint:TestPoint_Keystone_5010-5014_Multipurpose
- TP4: renamed from TP9; footprint (none) -> TestPoint:TestPoint_Keystone_5010-5014_Multipurpose
- TP5: renamed from TP10; footprint (none) -> TestPoint:TestPoint_Keystone_5010-5014_Multipurpose
- TP6: renamed from TP2; footprint (none) -> TestPoint:TestPoint_Keystone_5010-5014_Multipurpose
- TP7: renamed from TP11; footprint (none) -> TestPoint:TestPoint_Keystone_5010-5014_Multipurpose
- TP8: renamed from TP12; footprint (none) -> TestPoint:TestPoint_Keystone_5010-5014_Multipurpose
- TP9: renamed from TP1; footprint (none) -> TestPoint:TestPoint_Keystone_5010-5014_Multipurpose
- gave numbers to parts that had none: 3
- renumbered J4 to J5, J5 to J6, J6 to J7, U3 to U2, U4 to U3, U5 to U4, U2 to U5

Commit message: Inline calibration
Parts:
- C16: footprint Capacitor_SMD:C_0603_1608Metric_Pad1.08x0.95mm_HandSolder -> Capacitor_SMD:C_1206_3216Metric_Pad1.33x1.80mm_HandSolder
- JP1, JP2, JP3, JP4: footprint (none) -> Jumper:SolderJumper-3_P1.3mm_Open_RoundedPad1.0x1.5mm
- RV1, RV2, RV3, RV4: footprint (none) -> Potentiometer_SMD:Potentiometer_Bourns_3269W_Vertical
- U1, U2, U4, U5, U6: footprint (none) -> Package_SO:SOIC-8_3.9x4.9mm_P1.27mm
- U3: footprint (none) -> Package_SO:SOIC-16_3.9x9.9mm_P1.27mm
Changed lines of the file:
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@@
 			)
 		)
-		(property "Footprint" ""
+		(property "Footprint" "Package_SO:SOIC-8_3.9x4.9mm_P1.27mm"
 			(at 453.39 185.42 0)
 			(effects
@@
 			)
 		)
-		(property "Footprint" ""
+		(property "Footprint" "Package_SO:SOIC-8_3.9x4.9mm_P1.27mm"
 			(at 271.78 90.17 0)
 			(effects
@@
 			)
 		)
-		(property "Footprint" ""
+		(property "Footprint" "Package_SO:SOIC-8_3.9x4.9mm_P1.27mm"
 			(at 82.55 157.48 0)
 			(effects
@@
 			)
 		)
-		(property "Footprint" ""
+		(property "Footprint" "Package_SO:SOIC-8_3.9x4.9mm_P1.27mm"
 			(at 492.76 185.42 0)
 			(effects
@@
 			)
 		)
-		(property "Footprint" ""
+		(property "Footprint" "Package_SO:SOIC-8_3.9x4.9mm_P1.27mm"
 			(at 524.51 119.38 0)
 			(effects
@@
 			)
 		)
-		(property "Footprint" ""
+		(property "Footprint" "Package_SO:SOIC-8_3.9x4.9mm_P1.27mm"
 			(at 528.32 261.62 0)
 			(effects
@@
 			)
 		)
-		(property "Footprint" ""
+		(property "Footprint" "Potentiometer_SMD:Potentiometer_Bourns_3269W_Vertical"
 			(at 205.74 91.44 0)
 			(effects
@@
 			)
 		)
-		(property "Footprint" ""
+		(property "Footprint" "Jumper:SolderJumper-3_P1.3mm_Open_RoundedPad1.0x1.5mm"
 			(at 229.87 52.07 0)
 			(effects
@@
 			)
 		)
-		(property "Footprint" "Capacitor_SMD:C_0603_1608Metric_Pad1.08x0.95mm_HandSolder"
+		(property "Footprint" "Capacitor_SMD:C_1206_3216Metric_Pad1.33x1.80mm_HandSolder"
 			(at 124.1552 85.09 0)
 			(effects
@@
 			)
 		)
-		(property "Footprint" ""
+		(property "Footprint" "Package_SO:SOIC-8_3.9x4.9mm_P1.27mm"
 			(at 529.59 176.53 0)
 			(effects
@@
 			)
 		)
-		(property "Footprint" ""
+		(property "Footprint" "Jumper:SolderJumper-3_P1.3mm_Open_RoundedPad1.0x1.5mm"
 			(at 229.87 91.44 0)
 			(effects
@@
 			)
 		)
-		(property "Footprint" ""
+		(property "Footprint" "Package_SO:SOIC-8_3.9x4.9mm_P1.27mm"
 			(at 524.51 55.88 0)
 			(effects
@@
 			)
 		)
-		(property "Footprint" ""
+		(property "Footprint" "Jumper:SolderJumper-3_P1.3mm_Open_RoundedPad1.0x1.5mm"
 			(at 113.03 142.24 0)
 			(effects
@@
 			)
 		)
-		(property "Footprint" ""
+		(property "Footprint" "Potentiometer_SMD:Potentiometer_Bourns_3269W_Vertical"
 			(at 187.96 91.44 0)
 			(effects
@@
 			)
 		)
-		(property "Footprint" ""
+		(property "Footprint" "Potentiometer_SMD:Potentiometer_Bourns_3269W_Vertical"
 			(at 187.96 52.07 0)
 			(effects
@@
 			)
 		)
-		(property "Footprint" ""
+		(property "Footprint" "Potentiometer_SMD:Potentiometer_Bourns_3269W_Vertical"
 			(at 205.74 52.07 0)
 			(effects
@@
 			)
 		)
-		(property "Footprint" ""
+		(property "Footprint" "Package_SO:SOIC-8_3.9x4.9mm_P1.27mm"
 			(at 82.55 128.27 0)
 			(effects
@@
 			)
 		)
-		(property "Footprint" ""
+		(property "Footprint" "Package_SO:SOIC-8_3.9x4.9mm_P1.27mm"
 			(at 345.44 57.15 0)
 			(effects
@@
 			)
 		)
-		(property "Footprint" ""
+		(property "Footprint" "Package_SO:SOIC-8_3.9x4.9mm_P1.27mm"
 			(at 345.44 101.6 0)
 			(effects
@@
 			)
 		)
-		(property "Footprint" ""
+		(property "Footprint" "Package_SO:SOIC-16_3.9x9.9mm_P1.27mm"
 			(at 438.15 101.6 0)
 			(effects
@@
 			)
 		)
-		(property "Footprint" ""
+		(property "Footprint" "Package_SO:SOIC-8_3.9x4.9mm_P1.27mm"
 			(at 146.05 123.19 0)
 			(effects
@@
 			)
 		)
-		(property "Footprint" ""
+		(property "Footprint" "Package_SO:SOIC-8_3.9x4.9mm_P1.27mm"
 			(at 543.56 295.91 0)
 			(effects
@@
 			)
 		)
-		(property "Footprint" ""
+		(property "Footprint" "Package_SO:SOIC-8_3.9x4.9mm_P1.27mm"
 			(at 554.99 54.61 0)
 			(effects
@@
 			)
 		)
-		(property "Footprint" ""
+		(property "Footprint" "Jumper:SolderJumper-3_P1.3mm_Open_RoundedPad1.0x1.5mm"
 			(at 26.67 125.73 0)
 			(effects
@@
 			)
 		)
-		(property "Footprint" ""
+		(property "Footprint" "Package_SO:SOIC-8_3.9x4.9mm_P1.27mm"
 			(at 543.56 331.47 0)
 			(effects
